File: Kicad_Project/CCC_ESC.kicad_pcb (KiCad board)
At the start: 4 copper layers, 111.4 x 89.7 mm, 201 parts, among them J1 Conn_01x07, J2 Conn_01x06, J3 Conn_01x06, J4 Conn_01x06, SW1 Conn_01x02, U1 NCP5183 / TF2190-TAH, U2 NCP5183 / TF2190-TAH, U3 NCP5183 / TF2190-TAH, U4 NCS20034DR2G, U5 STM32F401CCU6_Balckpill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

Commit message: added in resistors, gate/source caps
Parts:
- added CSG1: C, Capacitor_SMD:C_0805_2012Metric, F.Cu at (53.4, 70.7)
- added CSG2: C, Capacitor_SMD:C_0805_2012Metric, F.Cu at (55.6, 87.7)
- added CSG3: C, Capacitor_SMD:C_0805_2012Metric, F.Cu at (85.9, 64.1)
- added CSG4: C, Capacitor_SMD:C_0805_2012Metric, F.Cu at (87.7, 86.6)
- added CSG5: C, Capacitor_SMD:C_0805_2012Metric, F.Cu at (118.3, 64.5)
- added CSG6: C, Capacitor_SMD:C_0805_2012Metric, F.Cu at (119.9, 86.5)
- added R42: R470, Resistor_SMD:R_0603_1608Metric, F.Cu at (94.8, 114.5)
- added R43: R470, Resistor_SMD:R_0603_1608Metric, F.Cu at (91.3, 114.5)
- added RN7: 470R, Resistor_SMD:R_Array_Concave_4x0603, F.Cu at (82.2, 115.2)
- moved R67 21.0 mm to (81.8, 98.2), turned to 0 degrees
- moved D9 16.4 mm to (81.8, 101.0), turned to -90 degrees
- moved CS2 5.40 mm to (85.7, 76.3), turned to -90 degrees
- moved CS3 4.95 mm to (118.3, 76.9), turned to -90 degrees
- moved CS1 4.19 mm to (53.6, 77.4), turned to -90 degrees
- moved RS1 2.82 mm to (53.6, 80.9), turned to -90 degrees
- moved RG10 2.25 mm to (85.7, 83.1)
- moved RS3 2.05 mm to (118.3, 80.3), turned to -90 degrees
- moved RG16 1.75 mm to (118.4, 83.8)
- moved RS2 1.63 mm to (85.7, 79.8), turned to -90 degrees
- moved C10 0.31 mm to (84.9, 115.2)
- moved C9 0.31 mm to (87.9, 115.2)
- moved C8 0.31 mm to (86.4, 115.2)
Connections:
- C19 pad 1: VSENSE -> GND
- C4 pad 1: VSENSE2 -> GND
- D4 pad 1: VSENSE2 -> VBAT
- D5 pad 1: VSENSE2 -> VBAT
- D6 pad 1: VSENSE2 -> VBAT
- R14 pad 1: VSENSE -> GND
- R15 pad 2: VSENSE -> GND
- R3 pad 1: VSENSE2 -> GND
- R38 pad 2: VSENSE -> GND
- R4 pad 2: VSENSE2 -> GND
- R40 pad 2: VSENSE2 -> GND
- U4 pad 13: VSENSE2 -> GND
- U5 pad 22: LIN_A -> _LIN_A
- U5 pad 23: LIN_B -> _LIN_B
- U5 pad 24: LIN_C -> _LIN_C
- U5 pad 25: HIN_A -> _HIN_A
- U5 pad 26: HIN_B -> _HIN_B
- U5 pad 27: HIN_C -> _HIN_C
- U5 pad 7: VSENSE -> GND
Routing:
- net GND: track 10.8 -> 195.9 mm, vias 338 -> 340
- net VSENSE2: track 109.3 -> 0.00 mm, vias 7 -> 3
- net VSENSE: track 74.9 -> 0.00 mm, vias 3 -> 0
- net HIN_B: track 33.8 -> 2.36 mm, vias 1 -> 0
- net _HIN_B: track 0.00 -> 31.3 mm, vias 0 -> 1
- net _HIN_A: track 0.00 -> 30.0 mm, vias 0 -> 1
- net HIN_A: track 34.9 -> 5.39 mm, vias 1 -> 2
- net HIN_C: track 26.3 -> 2.17 mm
- net A_SHA_V-: track 65.9 -> 42.1 mm, vias 3 -> 2
- net _HIN_C: track 0.00 -> 23.6 mm
- net A_SHA_V+: track 64.9 -> 41.8 mm, vias 3 -> 2
- net _LIN_A: track 0.00 -> 22.2 mm, vias 0 -> 1
- net _LIN_B: track 0.00 -> 21.5 mm, vias 0 -> 1
- net LIN_B: track 23.9 -> 2.55 mm, vias 1 -> 0
- net LIN_A: track 25.0 -> 5.20 mm, vias 1 -> 2
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Other:
- board size 111.4 x 89.7 mm -> 113.4 x 89.7 mm
- board text added: "Add gate to source capacitance - slow the MOS down if needed Reconsider expensive isolated gate drivers Diode between the DCDC and the gate driver 12V 470ohm resistors between pill and gate drivers"

Commit message: first draft
Parts:
- removed CSG1, CSG2, CSG3, CSG4, CSG5, CSG6: C, Capacitor_SMD:C_0805_2012Metric
- added CGS1: 6pF, Capacitor_SMD:C_0603_1608Metric, F.Cu at (53.4, 70.6)
- added CGS10: 6pF, Capacitor_SMD:C_0603_1608Metric, F.Cu at (55.1, 87.3)
- added CGS11: 6pF, Capacitor_SMD:C_0603_1608Metric, F.Cu at (64.4, 81.5)
- added CGS12: 6pF, Capacitor_SMD:C_0603_1608Metric, F.Cu at (74.6, 81.3)
- added CGS13: 6pF, Capacitor_SMD:C_0603_1608Metric, F.Cu at (88.1, 86.4)
- added CGS14: 6pF, Capacitor_SMD:C_0603_1608Metric, F.Cu at (96.6, 81.7)
- added CGS15: 6pF, Capacitor_SMD:C_0603_1608Metric, F.Cu at (106.9, 81.4)
- added CGS16: 6pF, Capacitor_SMD:C_0603_1608Metric, F.Cu at (119.8, 86.6)
- added CGS17: 6pF, Capacitor_SMD:C_0603_1608Metric, F.Cu at (129.2, 81.7)
- added CGS18: 6pF, Capacitor_SMD:C_0603_1608Metric, F.Cu at (139.5, 81.6)
- added CGS2: 6pF, Capacitor_SMD:C_0603_1608Metric, F.Cu at (64.2, 64.8)
- added CGS3: 6pF, Capacitor_SMD:C_0603_1608Metric, F.Cu at (74.5, 64.8)
- added CGS4: 6pF, Capacitor_SMD:C_0603_1608Metric, F.Cu at (85.9, 64.4)
- added CGS5: 6pF, Capacitor_SMD:C_0603_1608Metric, F.Cu at (96.5, 64.8)
- added CGS6: 6pF, Capacitor_SMD:C_0603_1608Metric, F.Cu at (106.9, 64.7)
- added CGS7: 6pF, Capacitor_SMD:C_0603_1608Metric, F.Cu at (118.3, 64.7)
- added CGS8: 6pF, Capacitor_SMD:C_0603_1608Metric, F.Cu at (128.9, 64.9)
- added CGS9: 6pF, Capacitor_SMD:C_0603_1608Metric, F.Cu at (139.2, 65.0)
- moved R22 3.51 mm to (116.4, 105.7), turned to 180 degrees
- moved R23 1.20 mm to (113.1, 106.3)
- moved RG10 0.77 mm to (85.9, 83.8), turned to -90 degrees
- moved R67 0.55 mm to (82.3, 98.2)
- moved U4 0.06 mm to (106.2, 108.3)
Connections:
- C19 pad 1: GND -> VSENSE
- C4 pad 1: GND -> VSENSE2
- D4 pad 1: VBAT -> VSENSE2
- D5 pad 1: VBAT -> VSENSE2
- D6 pad 1: VBAT -> VSENSE2
- QB2 pad 1: Net-(QB2-Pad1) -> Net-(CGS13-Pad1)
- R14 pad 1: GND -> VSENSE
- R15 pad 2: GND -> VSENSE
- R3 pad 1: GND -> VSENSE2
- R38 pad 2: GND -> VSENSE
- R4 pad 2: GND -> VSENSE2
- R40 pad 2: GND -> VSENSE2
- R50 pad 2: /BL_GATESIG -> Net-(U2-DRVL)
- RG10 pad 1: Net-(QB2-Pad1) -> Net-(U2-DRVL)
- RG10 pad 2: /BL_GATESIG -> Net-(CGS13-Pad1)
- RG11 pad 2: /BL_GATESIG -> Net-(U2-DRVL)
- RG12 pad 2: /BL_GATESIG -> Net-(U2-DRVL)
- U2 pad 4: /BL_GATESIG -> Net-(U2-DRVL)
- U4 pad 13: GND -> VSENSE2
- U5 pad 7: GND -> VSENSE
Routing:
- net GND: track 195.9 -> 12.5 mm, vias 340 -> 344
- net VSENSE2: track 0.00 -> 111.5 mm, vias 3 -> 7
- net VSENSE: track 0.00 -> 77.4 mm, vias 0 -> 3
- net Net-(U2-DRVL): track 0.00 -> 52.7 mm, vias 0 -> 3
- net /BL_GATESIG: track 41.6 -> 0.00 mm, vias 4 -> 0
- net PHASE_B: track 34.7 -> 57.0 mm, vias 67 -> 69
- net PHASE_A: track 34.5 -> 55.4 mm, vias 83 -> 79
- net A_SHA_V+: track 41.8 -> 62.0 mm
- net A_SHA_V-: track 42.1 -> 62.0 mm
- net /AL_GATESIG: track 44.4 -> 60.7 mm
- net PHASE_C: track 61.1 -> 76.5 mm, vias 69 -> 70
- net Net-(CGS16-Pad2): track 2.77 -> 12.4 mm, vias 0 -> 4
- net Net-(CGS10-Pad2): track 3.81 -> 13.0 mm, vias 0 -> 4
- net /CU_GATESIG: track 80.3 -> 87.8 mm
- net /CL_GATESIG: track 65.1 -> 71.7 mm, vias 4 -> 3
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
Commit message: first draft
Routing:
- net PHASE_C: vias 70 -> 86
- net PHASE_B: vias 69 -> 85
- net GND: vias 344 -> 338
Other:
- board text added: "Add gate to source capacitance - slow the MOS down if needed [DONE] Reconsider expensive isolated gate drivers [CAN DO] Diode between the DCDC and the gate driver 12V [NO PHYSICAL ROOM] 470ohm resistors between pill and gate drivers [DONE]"
- board text added: "Note masks for bus bars are on underside."
- board text added: "Use plastic washers with bolts -- could scrape through mask and _bang_."
- board text removed: "Add gate to source capacitance - slow the MOS down if needed Reconsider expensive isolated gate drivers Diode between the DCDC and the gate driver 12V 470ohm resistors between pill and gate drivers"
