File: Kicad_Project/CCC_ESC.kicad_pcb (KiCad board)
At the start: 4 copper layers, 113.9 x 90.3 mm, 221 parts, among them J1 Conn_01x07, J2 Conn_01x06, J3 Conn_01x06, J4 Conn_01x06, SW1 Conn_01x02, U1 NCP5183 / TF2190-TAH, U2 NCP5183 / TF2190-TAH, U3 NCP5183 / TF2190-TAH, U4 NCS20034DR2G, U5 STM32F401CCU6_Balckpill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

Commit message: minor touchups
Parts:
- moved CGS1 5.90 mm to (53.6, 64.5), turned to 90 degrees
- moved CGS13 1.64 mm to (89.4, 87.4), turned to -90 degrees
- moved CGS16 1.12 mm to (120.9, 87.6), turned to 90 degrees
- moved RG12 0.15 mm to (106.9, 84.6)
- moved PHA_2 0.11 mm to (76.1, 72.5)
- moved PHB_1 0.11 mm to (91.8, 72.5)
- moved PHB_2 0.11 mm to (108.3, 72.5)
Routing:
- net GND: track 33.4 -> 21.8 mm, vias 342 -> 347
- net Net-(CGS1-Pad2): track 6.30 -> 8.56 mm, vias 0 -> 2
- net A_SHA_V-: track 63.4 -> 62.2 mm
- net Net-(CGS16-Pad1): track 4.96 -> 6.02 mm, vias 0 -> 2
- net Net-(CGS13-Pad2): track 9.08 -> 9.92 mm
- net DV1H_N: track 78.1 -> 78.5 mm, vias 74 -> 60
- net DV3H_N: track 79.4 -> 79.2 mm, vias 77 -> 61
- net DV2H_N: track 59.4 -> 59.3 mm, vias 76 -> 60
Other:
- outline, holes or cut-outs redrawn
- board text added: "Top/bottom height of heat sink mount holes are assymetric."

Commit message: minor touchups
Routing:
- net GND: vias 347 -> 346
Other:
- board text added: "GND"
- board text added: "J1"
- board text added: "J2"
- board text added: "J3"
- board text added: "J4"
- board text added: "NEG"
- board text added: "NTC1"
- board text added: "POS"
- board text added: "Vcc"

Commit message: minor touchups
Parts:
- CGS1, CGS10, CGS11, CGS12, CGS13, CGS14, CGS15, CGS16, CGS17, CGS18, CGS2, CGS3, CGS4, CGS5, CGS6, CGS7, CGS8, CGS9: value 6nF -> 4.7nF
- moved PHB_2 0.19 mm to (108.5, 72.5)
- moved PHC_2 0.10 mm to (140.8, 72.5)
Connections:
- net /AL_GATESIG renamed DVRL1
- net /CL_GATESIG renamed DVRL3
- net Net-(U2-DRVL) renamed DVRL2
Routing:
- net DV3H_N: vias 61 -> 65
- net DV2H_N: vias 60 -> 59
Other:
- outline, holes or cut-outs redrawn
